File: DAOKI/DAOKI.kicad_pcb (KiCad board)
At the start: 2 copper layers, 14 parts, among them CON4 CON4, U1 MOCH22a1, U2 LM393

Commit message: adding PCB
Parts:
- D2: footprint Resistor_SMD:R_0603_1608Metric_Pad0.98x0.95mm_HandSolder -> LED_SMD:LED_0603_1608Metric_Pad1.05x0.95mm_HandSolder
- R4: value 1K -> 100
- moved R3 45.9 mm to (157.0, 95.0), turned to 270 degrees
- moved U2 44.7 mm to (159.0, 103.0), turned to 180 degrees
- moved R6 36.4 mm to (150.1, 100.0)
- moved CON4 33.9 mm to (177.0, 94.0)
- moved R4 31.7 mm to (150.1, 103.0), turned to 180 degrees
- moved R7 31.6 mm to (167.0, 101.0), turned to 90 degrees
- moved U1 31.3 mm to (139.0, 93.8)
- moved R1 28.7 mm to (167.0, 95.0), turned to 270 degrees
- moved C1 27.8 mm to (150.0, 91.0)
- moved C2 24.3 mm to (150.0, 94.0), turned to 180 degrees
- moved R5 23.3 mm to (149.9, 97.0)
- moved D2 20.0 mm to (172.0, 102.0)
- moved R2 19.5 mm to (162.0, 95.0), turned to 270 degrees
- moved D1 17.1 mm to (172.0, 94.0)
Routing:
- net +5V: track 0.00 -> 68.2 mm
- net GND: track 0.00 -> 62.7 mm, vias 0 -> 3
- net Net-(C2-Pad1): track 0.00 -> 52.2 mm, vias 0 -> 1
- net Net-(CON4-Pad3): track 0.00 -> 32.6 mm, vias 0 -> 1
- net Net-(R4-Pad2): track 0.00 -> 23.9 mm, vias 0 -> 1
- net Net-(R2-Pad1): track 0.00 -> 14.1 mm
- net Net-(D2-Pad1): track 0.00 -> 4.16 mm
- net Net-(D1-Pad1): track 0.00 -> 4.16 mm
- added copper zone on F.Cu, net +5V
- added copper zone on B.Cu, net GND
Other:
- net class Default: clearance 0.2 -> 0.3; trace_width 0.25 -> 0.8; via_dia 0.8 -> 1.6; via_drill 0.4 -> 0.8
- rule trace_clearance: 0.2 -> 0.3
